File: ECG/ECG.brd (EAGLE design)
At the start: 100 x 80 mm, 36 parts, among them J1 TC2030-CTX-NL, U1 BGM111-VISUAL-A, U2 AD8232

Commit message: Initial Layout for the Board
Parts:
- moved R25 120.9 mm to (66.0, 68.6), turned to 270 degrees
- moved R35 120.3 mm to (68.6, 77.5)
- moved JP5 112.4 mm to (71.1, 69.8), turned to 270 degrees
- moved C11 106.0 mm to (49.5, 77.5), turned to 270 degrees
- moved R23 100.7 mm to (54.6, 58.4)
- moved R24 99.5 mm to (47.0, 73.7)
- moved R32 99.5 mm to (61.0, 63.5), turned to 270 degrees
- moved R33 96.5 mm to (54.6, 54.6)
- moved C13 95.4 mm to (64.8, 54.6), turned to 180 degrees
- moved R31 95.2 mm to (58.4, 76.2), turned to 180 degrees
- moved C14 94.1 mm to (59.7, 54.6), turned to 180 degrees
- moved R34 93.0 mm to (47.0, 62.2)
- moved R37 93.0 mm to (36.8, 77.5), turned to 90 degrees
- moved JP6 92.2 mm to (44.5, 54.6)
- moved C9 90.2 mm to (66.0, 64.8), turned to 180 degrees
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