File: ECG/ECG_V5.brd (EAGLE design)
At the start: 62.2 x 34.3 mm, 35 parts, among them U1 AD8232, U3 BGM111-VISUAL-A

Commit message: Moved BGM111
Parts:
- moved SJ1 7.91 mm to (9.14, 43.1), turned to 180 degrees
- moved D2 5.86 mm to (7.75, 40.0), turned to 270 degrees
- moved R39 5.36 mm to (8.00, 36.8)
- moved U3 3.18 mm to (23.7, 41.5)
Routing:
- net SIGNAL_OUT: track 105.6 -> 90.5 mm, vias 8 -> 7
- net N$37: track 13.1 -> 3.43 mm
- net GND: track 124.0 -> 131.6 mm
- net N$36: track 9.16 -> 3.33 mm
- net N$31: track 23.0 -> 26.1 mm
- net 3.3V: track 72.1 -> 75.2 mm
- net N$33: track 21.2 -> 23.3 mm
- net N$29: track 34.8 -> 35.8 mm
