File: EEG-EMG/EEG-EMG_V1.sch (EAGLE design)
At the start: 62 parts, among them IC1 MCP6V31, IC11 LM7332MA, IC2 MCP6V31, IC3 MCP6V31, IC4 MCP6V31, IC6 MCP3912, Q7 CSM-3X-CRYSTALCSM-3X, U2 BGM111-VISUAL-A

Commit message: SPI Connections Done
Connections:
- new net N$28: IC6.SDO, U2.PC7
- new net N$29: IC6.SCK, U2.PC8
- new net N$30: IC6.CS*, U2.PC9
- net N$27: now also IC6.SDI, U2.PC6; no longer IC6.SDO, U2.PB11
- net VAA: no longer IC6.DVDD
Changed lines of the file:
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@@
 </segment>
 <segment>
-<pinref part="IC6" gate="G$1" pin="DVDD"/>
-<wire x1="878.84" y1="-78.74" x2="881.38" y2="-78.74" width="0.1524" layer="91"/>
 <pinref part="C45" gate="G$1" pin="2"/>
 <wire x1="881.38" y1="-78.74" x2="937.26" y2="-78.74" width="0.1524" layer="91"/>
 <wire x1="937.26" y1="-78.74" x2="937.26" y2="-86.36" width="0.1524" layer="91"/>
-<junction x="881.38" y="-78.74"/>
 <wire x1="881.38" y1="-78.74" x2="881.38" y2="-68.58" width="0.1524" layer="91"/>
 <wire x1="881.38" y1="-68.58" x2="883.92" y2="-68.58" width="0.1524" layer="91"/>
@@
 <net name="N$27" class="0">
 <segment>
+<pinref part="IC6" gate="G$1" pin="SDI"/>
+<wire x1="878.84" y1="-83.82" x2="949.96" y2="-83.82" width="0.1524" layer="91"/>
+<wire x1="949.96" y1="-83.82" x2="949.96" y2="-220.98" width="0.1524" layer="91"/>
+<wire x1="949.96" y1="-220.98" x2="960.12" y2="-220.98" width="0.1524" layer="91"/>
+<wire x1="960.12" y1="-220.98" x2="960.12" y2="-218.44" width="0.1524" layer="91"/>
+<wire x1="960.12" y1="-218.44" x2="1008.38" y2="-218.44" width="0.1524" layer="91"/>
+<wire x1="1008.38" y1="-218.44" x2="1008.38" y2="-220.98" width="0.1524" layer="91"/>
+<pinref part="U2" gate="G$1" pin="PC6"/>
+<wire x1="1008.38" y1="-220.98" x2="1018.54" y2="-220.98" width="0.1524" layer="91"/>
+<wire x1="1018.54" y1="-220.98" x2="1018.54" y2="-218.44" width="0.1524" layer="91"/>
+</segment>
+</net>
+<net name="N$28" class="0">
+<segment>
 <pinref part="IC6" gate="G$1" pin="SDO"/>
 <wire x1="878.84" y1="-86.36" x2="955.04" y2="-86.36" width="0.1524" layer="91"/>
-<wire x1="955.04" y1="-86.36" x2="955.04" y2="-203.2" width="0.1524" layer="91"/>
-<pinref part="U2" gate="G$1" pin="PB11"/>
-<wire x1="955.04" y1="-203.2" x2="1005.84" y2="-203.2" width="0.1524" layer="91"/>
-</segment>
-</net>
+<wire x1="955.04" y1="-86.36" x2="955.04" y2="-223.52" width="0.1524" layer="91"/>
+<wire x1="955.04" y1="-223.52" x2="962.66" y2="-223.52" width="0.1524" layer="91"/>
+<wire x1="962.66" y1="-223.52" x2="962.66" y2="-220.98" width="0.1524" layer="91"/>
+<wire x1="962.66" y1="-220.98" x2="965.2" y2="-220.98" width="0.1524" layer="91"/>
+<wire x1="965.2" y1="-220.98" x2="965.2" y2="-213.36" width="0.1524" layer="91"/>
+<wire x1="965.2" y1="-213.36" x2="1000.76" y2="-213.36" width="0.1524" layer="91"/>
+<wire x1="1000.76" y1="-213.36" x2="1000.76" y2="-223.52" width="0.1524" layer="91"/>
+<pinref part="U2" gate="G$1" pin="PC7"/>
+<wire x1="1000.76" y1="-223.52" x2="1021.08" y2="-223.52" width="0.1524" layer="91"/>
+<wire x1="1021.08" y1="-223.52" x2="1021.08" y2="-218.44" width="0.1524" layer="91"/>
+</segment>
+</net>
+<net name="N$29" class="0">
+<segment>
+<pinref part="IC6" gate="G$1" pin="SCK"/>
+<wire x1="878.84" y1="-88.9" x2="957.58" y2="-88.9" width="0.1524" layer="91"/>
+<wire x1="957.58" y1="-88.9" x2="957.58" y2="-91.44" width="0.1524" layer="91"/>
+<wire x1="957.58" y1="-91.44" x2="965.2" y2="-91.44" width="0.1524" layer="91"/>
+<wire x1="965.2" y1="-91.44" x2="965.2" y2="-259.08" width="0.1524" layer="91"/>
+<pinref part="U2" gate="G$1" pin="PC8"/>
+<wire x1="965.2" y1="-259.08" x2="1023.62" y2="-259.08" width="0.1524" layer="91"/>
+<wire x1="1023.62" y1="-259.08" x2="1023.62" y2="-218.44" width="0.1524" layer="91"/>
+</segment>
+</net>
+<net name="N$30" class="0">
+<segment>
+<wire x1="970.28" y1="-81.28" x2="970.28" y2="-200.66" width="0.1524" layer="91"/>
+<wire x1="970.28" y1="-200.66" x2="942.34" y2="-200.66" width="0.1524" layer="91"/>
+<wire x1="942.34" y1="-200.66" x2="942.34" y2="-271.78" width="0.1524" layer="91"/>
+<pinref part="U2" gate="G$1" pin="PC9"/>
+<wire x1="942.34" y1="-271.78" x2="1026.16" y2="-271.78" width="0.1524" layer="91"/>
+<wire x1="1026.16" y1="-271.78" x2="1026.16" y2="-218.44" width="0.1524" layer="91"/>
+<pinref part="IC6" gate="G$1" pin="CS*"/>
+<wire x1="878.84" y1="-91.44" x2="952.5" y2="-91.44" width="0.1524" layer="91"/>
+<wire x1="952.5" y1="-91.44" x2="952.5" y2="-81.28" width="0.1524" layer="91"/>
+<wire x1="952.5" y1="-81.28" x2="970.28" y2="-81.28" width="0.1524" layer="91"/>
+</segment>
+</net>

Commit message: Changed EMG Jumper Connection
Parts:
- removed BAT1: 2032, SMTU-2032-1:2032
- removed JP2: (no value), jumper:JP2Q
- added JP3: (no value), jumper:JP2E
Connections:
- removed net EMG1-: IA_3.IN-, JP2.2
- removed net EMG2-: IA_4.IN-, JP2.4
- net EMG1+: now also JP3.1; no longer JP2.1
- net EMG2+: now also JP3.2; no longer JP2.3
- net GND: no longer BAT1.-
- net REF: now also IA_3.IN-, IA_4.IN-, JP3.3
- net VAA: now also BAT2.+, IC6.DVDD; no longer BAT1.+
- net VDD: no longer BAT2.+
Other:
- moved on the sheet: BAT2

Commit message: Completed Board - Basic Functionality V1
Parts:
- removed JP3: (no value), jumper:JP2E
- added JP2: (no value), jumper:JP2W
Connections:
- net EMG1+: now also JP2.1; no longer JP3.1
- net EMG2+: now also JP2.2; no longer JP3.2
- net REF: now also JP2.3; no longer JP3.3
Changed lines of the file:
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@@
 <part name="GND29" library="SparkFun-Aesthetics" deviceset="GND" device=""/>
 <part name="J2" library="tag-connect" deviceset="TC2030" device="-MCP-NL"/>
-<part name="JP3" library="jumper" deviceset="JP2E" device=""/>
 <part name="BAT2" library="SMTU-2032-1" deviceset="2032" device=""/>
+<part name="JP2" library="jumper" deviceset="JP2W" device=""/>
 </parts>
 <sheets>
@@
 <instance part="GND29" gate="1" x="1013.46" y="-233.68"/>
 <instance part="J2" gate="G$1" x="982.98" y="-228.6" rot="R180"/>
-<instance part="JP3" gate="1" x="383.54" y="-299.72"/>
 <instance part="BAT2" gate="G$1" x="381" y="-43.18" rot="R180"/>
+<instance part="JP2" gate="1" x="383.54" y="-289.56"/>
 </instances>
 <busses>
@@
 <wire x1="472.44" y1="-299.72" x2="472.44" y2="-312.42" width="0.1524" layer="91"/>
 <wire x1="472.44" y1="-312.42" x2="381" y2="-312.42" width="0.1524" layer="91"/>
-<pinref part="JP3" gate="1" pin="1"/>
-<wire x1="381" y1="-302.26" x2="381" y2="-312.42" width="0.1524" layer="91"/>
+<pinref part="JP2" gate="1" pin="1"/>
+<wire x1="381" y1="-292.1" x2="381" y2="-312.42" width="0.1524" layer="91"/>
 </segment>
 </net>
@@
 <wire x1="398.78" y1="-307.34" x2="398.78" y2="-429.26" width="0.1524" layer="91"/>
 <wire x1="398.78" y1="-429.26" x2="497.84" y2="-429.26" width="0.1524" layer="91"/>
-<pinref part="JP3" gate="1" pin="2"/>
 <wire x1="398.78" y1="-307.34" x2="383.54" y2="-307.34" width="0.1524" layer="91"/>
-<wire x1="383.54" y1="-307.34" x2="383.54" y2="-302.26" width="0.1524" layer="91"/>
+<pinref part="JP2" gate="1" pin="2"/>
+<wire x1="383.54" y1="-292.1" x2="383.54" y2="-307.34" width="0.1524" layer="91"/>
 </segment>
 </net>
@@
 <wire x1="391.16" y1="-177.8" x2="391.16" y2="-292.1" width="0.1524" layer="91"/>
 <junction x="439.42" y="-177.8"/>
-<pinref part="JP3" gate="1" pin="3"/>
 <wire x1="391.16" y1="-292.1" x2="391.16" y2="-299.72" width="0.1524" layer="91"/>
 <wire x1="391.16" y1="-299.72" x2="391.16" y2="-302.26" width="0.1524" layer="91"/>
@@
 <wire x1="398.78" y1="-299.72" x2="391.16" y2="-299.72" width="0.1524" layer="91"/>
 <junction x="391.16" y="-299.72"/>
-</segment>
-</net>
+<pinref part="JP2" gate="1" pin="3"/>
+<wire x1="386.08" y1="-292.1" x2="386.08" y2="-302.26" width="0.1524" layer="91"/>
+</segment>
+</net>
