File: EEG-EMG/EEG-EMG_V1.brd (EAGLE design)
At the start: 106 x 40.6 mm, 62 parts, among them IC1 MCP6V31, IC11 LM7332MA, IC2 MCP6V31, IC3 MCP6V31, IC4 MCP6V31, IC6 MCP3912, Q7 CSM-3X-CRYSTALCSM-3X, U2 BGM111-VISUAL-A

Commit message: Completed Board - Basic Functionality V1
Parts:
- removed BAT1: 2032, SMTU-2032-1:KZH20SMD
- JP2: device jumper:JP2Q -> jumper:JP2W
- moved BAT2 33.0 mm to (44.5, 63.5)
- moved JP2 2.54 mm to (3.81, 57.1), turned to 0 degrees
Connections:
- removed net EMG1-: IA_3.P3, JP2.2
- removed net EMG2-: IA_4.P3, JP2.4
- new net N$28: IC6.25, U2.PC7
- new net N$29: IC6.24, U2.PC8
- new net N$30: IC6.23, U2.PC9
- net EMG2+: now also JP2.2; no longer JP2.3
- net GND: no longer BAT1.-
- net N$27: now also IC6.26, U2.PC6; no longer IC6.25, U2.PB11
- net REF: now also IA_3.P3, IA_4.P3, JP2.3
- net VAA: now also BAT2.+; no longer BAT1.+
- net VDD: no longer BAT2.+
Routing:
- net REF: track 29.6 -> 89.8 mm, vias 0 -> 2
- net VDD: track 38.1 -> 15.5 mm, vias 3 -> 2
- net N$30: track 0.00 -> 20.9 mm, vias 0 -> 2
- net N$29: track 0.00 -> 19.6 mm, vias 0 -> 2
- net EMG2-: track 18.4 -> 0.00 mm
- net N$28: track 0.00 -> 18.2 mm, vias 0 -> 2
- net EMG1-: track 16.3 -> 0.00 mm
- net GND: track 365.1 -> 350.5 mm
- net EMG1+: track 23.9 -> 34.1 mm, vias 0 -> 1
- net VAA: track 242.0 -> 250.8 mm
- net EMG2+: track 27.1 -> 30.9 mm, vias 0 -> 1
- net N$27: track 18.4 -> 17.2 mm
